File: hardware/board.brd (EAGLE design)
At the start: 75.9 x 21.7 mm, 17 parts, among them IC1 MCP4131, IC2 L272, Q1 BC638, Q3 BC638

Commit message: renaming things, adding images
Other:
- board text added: "Whistle Board Version 1"
- board text removed: "Branding Goes Here V1 underdogma.net/trains"
Changed lines of the file:
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@@
 <setting verticaltext="up"/>
 </settings>
-<grid distance="0.005" unitdist="inch" unit="inch" style="lines" multiple="1" display="yes" altdistance="0.025" altunitdist="inch" altunit="inch"/>
+<grid distance="0.05" unitdist="inch" unit="inch" style="lines" multiple="1" display="yes" altdistance="0.025" altunitdist="inch" altunit="inch"/>
 <layers>
 <layer number="1" name="Top" color="4" fill="1" visible="yes" active="yes"/>
@@
 <layer number="49" name="Reference" color="7" fill="1" visible="yes" active="yes"/>
 <layer number="50" name="dxf" color="7" fill="1" visible="no" active="no"/>
-<layer number="51" name="tDocu" color="7" fill="1" visible="no" active="yes"/>
+<layer number="51" name="tDocu" color="7" fill="1" visible="yes" active="yes"/>
 <layer number="52" name="bDocu" color="7" fill="1" visible="yes" active="yes"/>
 <layer number="53" name="tGND_GNDA" color="7" fill="9" visible="no" active="no"/>
@@
 <wire x1="65.024" y1="1.7145" x2="61.595" y2="1.7145" width="0.8128" layer="30" curve="-165.227914"/>
 <wire x1="60.0075" y1="1.7145" x2="56.5785" y2="1.7145" width="0.8128" layer="30" curve="-165.227914"/>
-<text x="46.99" y="4.699" size="1.016" layer="22" rot="MR0">Branding Goes Here V1
-underdogma.net/trains</text>
+<text x="46.99" y="4.699" size="1.016" layer="22" rot="MR0">Whistle Board
+Version 1</text>
 </plain>
 <attributes>
@@
 <contactref element="IC1" pad="V+"/>
 <polygon width="0.254" layer="1" isolate="0.3048">
-<vertex x="-4.2926" y="23.114"/>
-<vertex x="82.1436" y="23.114"/>
-<vertex x="82.1436" y="6.3246"/>
-<vertex x="82.1436" y="-3.556"/>
-<vertex x="-5.2578" y="-3.556"/>
-<vertex x="-5.2578" y="23.0886"/>
-<vertex x="-4.2926" y="23.0886"/>
+<vertex x="0.0254" y="21.844"/>
+<vertex x="75.4126" y="21.844"/>
+<vertex x="75.4126" y="0"/>
+<vertex x="-0.0508" y="0.127"/>
+<vertex x="-0.0508" y="21.8186"/>
+<vertex x="0.1524" y="21.8186"/>
 </polygon>
 <contactref element="R1" pad="P$1"/>
@@
 </signal>
 <signal name="GND">
-<polygon width="0.254" layer="16">
-<vertex x="0" y="0.1524"/>
-<vertex x="0" y="23.0124"/>
-<vertex x="79.0956" y="23.0124" curve="90"/>
-<vertex x="79.248" y="23.1648"/>
-<vertex x="79.248" y="0.1524"/>
-</polygon>
 <contactref element="S1" pad="NO1"/>
 <contactref element="S1" pad="NC2"/>
@@
 <contactref element="POW" pad="2"/>
 <contactref element="AUX" pad="2"/>
+<polygon width="0.4064" layer="16">
+<vertex x="0" y="0"/>
+<vertex x="0" y="21.59"/>
+<vertex x="60.96" y="21.59"/>
+<vertex x="76.2" y="21.59"/>
+<vertex x="76.2" y="0"/>
+</polygon>
 </signal>
 <signal name="EN">
