File: hardware/supply.brd (EAGLE design)
At the start: 25.4 x 53.3 mm, 14 parts

Commit message: renaming things, adding images
Parts:
- removed JP1: POWER_JACKPTH, SparkFun-Connectors:POWER_JACK_PTH
- added V5: POWER_JACKPTH, SparkFun-Connectors:POWER_JACK_PTH
- moved R1 1.27 mm to (19.7, 36.8)
- renumbered JP2 to V+, JP3 to MC, JP4 to B1, JP5 to B2, JP6 to B3
Connections:
- net 5V: now also V5.PWR; no longer JP1.PWR
- net GND: now also V5.GND; no longer JP1.GND
Routing:
- net V+: track 30.5 -> 29.4 mm
- net N$4: track 8.92 -> 9.46 mm
Other:
- board text added: "Whistle Supply Version 1"
Changed lines of the file:
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@@
 <hole x="26.67" y="47.625" drill="3.2"/>
 <hole x="8.89" y="10.795" drill="3.2"/>
+<text x="22.225" y="42.545" size="1.016" layer="22" rot="MR0">Whistle Supply
+Version 1</text>
 </plain>
 <attributes>
@@
 </autorouter>
 <elements>
-<element name="JP1" library="SparkFun-Connectors" package="POWER_JACK_PTH" value="POWER_JACKPTH" x="0.635" y="38.735" rot="R270">
-<attribute name="PROD_ID" value="CONN-08197" x="0.635" y="38.735" size="1.778" layer="27" rot="R270" display="off"/>
-</element>
-<element name="JP2" library="SparkFun-Connectors" package="SCREWTERMINAL-5MM-2" value="" x="7.62" y="22.225" rot="R270">
+<element name="V5" library="SparkFun-Connectors" package="POWER_JACK_PTH" value="POWER_JACKPTH" x="1.27" y="38.735" rot="R270">
+<attribute name="PROD_ID" value="CONN-08197" x="1.27" y="38.735" size="1.778" layer="27" rot="R270" display="off"/>
+</element>
+<element name="V+" library="SparkFun-Connectors" package="SCREWTERMINAL-5MM-2" value="" x="7.62" y="22.225" rot="R270">
 <attribute name="STOREFRONT_ID" value="PRT-08432" x="7.62" y="22.225" size="1.778" layer="27" rot="R270" display="off"/>
 </element>
 <element name="U$1" library="custom-parts" package="3KBP0X" value="3KBP0X" x="21.59" y="31.75" rot="R180"/>
-<element name="R1" library="SparkFun-Resistors" package="AXIAL-0.3EZ" value="330" x="18.415" y="36.83" rot="R90">
-<attribute name="PROD_ID" value="RES-08380" x="18.415" y="36.83" size="1.778" layer="27" rot="R90" display="off"/>
+<element name="R1" library="SparkFun-Resistors" package="AXIAL-0.3EZ" value="330" x="19.685" y="36.83" rot="R90">
+<attribute name="PROD_ID" value="RES-08380" x="19.685" y="36.83" size="1.778" layer="27" rot="R90" display="off"/>
 </element>
 <element name="R3" library="SparkFun-Resistors" package="AXIAL-0.3EZ" value="270" x="17.78" y="22.225" rot="R180">
@@
 <element name="D3" library="SparkFun-LED" package="LED10MM" value="" x="17.78" y="48.26" rot="R180"/>
 <element name="D4" library="SparkFun-LED" package="LED10MM" value="" x="17.78" y="10.16" rot="R180"/>
-<element name="JP4" library="SparkFun-Connectors" package="1X03" value="" x="27.305" y="29.21" rot="R90"/>
-<element name="JP3" library="SparkFun-Connectors" package="1X02" value="" x="27.305" y="39.37" rot="R90"/>
-<element name="JP5" library="SparkFun-Connectors" package="1X03" value="" x="27.305" y="20.955" rot="R90"/>
-<element name="JP6" library="SparkFun-Connectors" package="1X03" value="" x="27.305" y="12.7" rot="R90"/>
+<element name="B1" library="SparkFun-Connectors" package="1X03" value="" x="27.305" y="29.21" rot="R90"/>
+<element name="MC" library="SparkFun-Connectors" package="1X02" value="" x="27.305" y="39.37" rot="R90"/>
+<element name="B2" library="SparkFun-Connectors" package="1X03" value="" x="27.305" y="20.955" rot="R90"/>
+<element name="B3" library="SparkFun-Connectors" package="1X03" value="" x="27.305" y="12.7" rot="R90"/>
 </elements>
 <signals>
 <signal name="I1">
 <contactref element="U$1" pad="I1"/>
-<contactref element="JP2" pad="2"/>
+<contactref element="V+" pad="2"/>
 <wire x1="7.62" y1="17.225" x2="10.16" y2="19.765" width="0.8128" layer="1"/>
 <wire x1="10.16" y1="19.765" x2="10.16" y2="24.024790625" width="0.8128" layer="1"/>
@@
 <signal name="I2">
 <contactref element="U$1" pad="I2"/>
-<contactref element="JP2" pad="1"/>
+<contactref element="V+" pad="1"/>
 <wire x1="7.62" y1="22.225" x2="7.62" y2="25.08" width="0.8128" layer="1"/>
 <wire x1="7.62" y1="25.08" x2="11.89" y2="29.35" width="0.8128" layer="1"/>
@@
 <signal name="5V">
 <contactref element="R1" pad="P$1"/>
-<contactref element="JP1" pad="PWR"/>
+<contactref element="V5" pad="PWR"/>
 <polygon width="0.8128" layer="1" isolate="0.6096">
-<vertex x="0" y="32.385"/>
-<vertex x="37.465" y="32.385"/>
-<vertex x="37.465" y="59.055"/>
-<vertex x="0" y="59.055"/>
+<vertex x="5.08" y="32.385"/>
+<vertex x="30.48" y="32.385"/>
+<vertex x="30.48" y="55.88"/>
+<vertex x="5.08" y="55.88"/>
 </polygon>
-<contactref element="JP4" pad="1"/>
-<contactref element="JP3" pad="2"/>
-<contactref element="JP5" pad="1"/>
-<contactref element="JP6" pad="1"/>
+<contactref element="B1" pad="1"/>
+<contactref element="MC" pad="2"/>
+<contactref element="B2" pad="1"/>
+<contactref element="B3" pad="1"/>
 <wire x1="27.305" y1="12.7" x2="29.13560625" y2="14.53060625" width="0.254" layer="1"/>
 <wire x1="29.13560625" y1="14.53060625" x2="29.21" y2="14.710209375" width="0.254" layer="1" curve="44.999295"/>
@@
 <signal name="GND">
 <contactref element="U$1" pad="-"/>
-<contactref element="JP1" pad="GND"/>
+<contactref element="V5" pad="GND"/>
 <polygon width="0.4064" layer="16">
-<vertex x="0" y="0"/>
-<vertex x="0" y="80.01"/>
-<vertex x="100.33" y="80.01"/>
-<vertex x="100.33" y="0"/>
+<vertex x="5.08" y="2.54"/>
+<vertex x="5.08" y="55.88"/>
+<vertex x="30.48" y="55.88"/>
+<vertex x="30.48" y="2.54"/>
 </polygon>
 <contactref element="D4" pad="C"/>
 <contactref element="D3" pad="C"/>
-<contactref element="JP4" pad="2"/>
-<contactref element="JP3" pad="1"/>
-<contactref element="JP5" pad="2"/>
-<contactref element="JP6" pad="2"/>
+<contactref element="B1" pad="2"/>
+<contactref element="MC" pad="1"/>
+<contactref element="B2" pad="2"/>
+<contactref element="B3" pad="2"/>
 </signal>
 <signal name="V+">
 <contactref element="U$1" pad="+"/>
-<contactref element="JP4" pad="3"/>
+<contactref element="B1" pad="3"/>
 <contactref element="R2" pad="P$1"/>
-<contactref element="JP5" pad="3"/>
-<contactref element="JP6" pad="3"/>
+<contactref element="B2" pad="3"/>
+<contactref element="B3" pad="3"/>
 <wire x1="27.305" y1="34.29" x2="24.20439375" y2="31.18939375" width="0.8128" layer="1"/>
 <wire x1="24.20439375" y1="31.18939375" x2="24.13" y2="31.009790625" width="0.8128" layer="1" curve="44.999295"/>
-<wire x1="24.13" y1="31.009790625" x2="24.13" y2="24.765" width="0.8128" layer="1"/>
+<wire x1="24.13" y1="31.009790625" x2="24.13" y2="29.35" width="0.8128" layer="1"/>
+<wire x1="24.13" y1="29.35" x2="24.13" y2="24.765" width="0.8128" layer="1"/>
 <wire x1="24.13" y1="24.765" x2="24.13" y2="21.060209375" width="0.8128" layer="1"/>
 <wire x1="24.13" y1="21.060209375" x2="24.20439375" y2="20.88060625" width="0.8128" layer="1" curve="44.999502"/>
 <wire x1="24.20439375" y1="20.88060625" x2="27.305" y2="17.78" width="0.8128" layer="1"/>
-<wire x1="21.59" y1="24.765" x2="24.13" y2="24.765" width="0.8128" layer="1"/>
 <wire x1="24.13" y1="24.765" x2="25.32560625" y2="25.96060625" width="0.8128" layer="1"/>
 <wire x1="25.32560625" y1="25.96060625" x2="25.505209375" y2="26.035" width="0.8128" layer="1" curve="-44.999295"/>
 <wire x1="25.505209375" y1="26.035" x2="27.305" y2="26.035" width="0.8128" layer="1"/>
-<wire x1="20.09" y1="29.35" x2="21.51560625" y2="27.92439375" width="0.8128" layer="1"/>
-<wire x1="21.51560625" y1="27.92439375" x2="21.59" y2="27.744790625" width="0.8128" layer="1" curve="-44.999295"/>
-<wire x1="21.59" y1="27.744790625" x2="21.59" y2="24.765" width="0.8128" layer="1"/>
+<wire x1="20.09" y1="29.35" x2="24.13" y2="29.35" width="0.8128" layer="1"/>
+<wire x1="21.59" y1="24.765" x2="24.13" y2="24.765" width="0.254" layer="1"/>
 </signal>
 <signal name="N$4">
 <contactref element="R1" pad="P$2"/>
 <contactref element="D3" pad="A"/>
-<wire x1="18.415" y1="40.64" x2="15.31439375" y2="43.74060625" width="0.254" layer="1"/>
-<wire x1="15.31439375" y1="43.74060625" x2="15.24" y2="43.920209375" width="0.254" layer="1" curve="-44.999295"/>
-<wire x1="15.24" y1="43.920209375" x2="15.24" y2="48.26" width="0.254" layer="1"/>
+<wire x1="15.24" y1="48.26" x2="15.24" y2="45.085" width="0.254" layer="1"/>
+<wire x1="15.24" y1="45.085" x2="19.685" y2="40.64" width="0.254" layer="1"/>
 </signal>
 <signal name="N$1">
@@
 </board>
 </drawing>
+<compatibility>
+<note version="6.3" minversion="6.2.2" severity="warning">
+Since Version 6.2.2 text objects can contain more than one line,
+which will not be processed correctly with this version.
+</note>
+</compatibility>
 </eagle>
