File: hardware/whistle-board.brd (EAGLE design)
At the start: 75.9 x 21.7 mm, 15 parts, among them IC1 MCP4131, IC2 L272

Commit message: Updating license, annotating schematic, updating images, moving software
Parts:
- added FRAME1: FRAME-LETTER, SparkFun-Aesthetics:CREATIVE_COMMONS
Connections:
- net 12V renamed VCC
Changed lines of the file:
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@@
 <element name="AUX" library="SparkFun-Connectors" package="1X02" value="" x="57.15" y="17.145" rot="R180"/>
 <element name="D2" library="SparkFun-DiscreteSemi" package="DIODE-1N4001" value="" x="49.657" y="12.065" rot="R90"/>
+<element name="FRAME1" library="SparkFun-Aesthetics" package="CREATIVE_COMMONS" value="FRAME-LETTER" x="20.4216" y="-7.6708"/>
 </elements>
 <signals>
@@
 <contactref element="IC2" pad="IN2-"/>
 <contactref element="AUX" pad="1"/>
-</signal>
-<signal name="12V">
-<contactref element="POW" pad="1"/>
-<contactref element="IC2" pad="V+"/>
-<wire x1="35.2679" y1="9.8425" x2="35.2679" y2="11.1379" width="0.508" layer="1"/>
-<wire x1="35.2679" y1="11.1379" x2="39.37" y2="15.24" width="0.508" layer="1"/>
-<wire x1="39.37" y1="15.24" x2="39.37" y2="17.145" width="0.508" layer="1"/>
 </signal>
 <signal name="SDI">
@@
 <wire x1="45.5168" y1="6.985" x2="49.657" y2="6.985" width="0.508" layer="1"/>
 </signal>
+<signal name="VCC">
+<contactref element="POW" pad="1"/>
+<contactref element="IC2" pad="V+"/>
+<wire x1="35.2679" y1="9.8425" x2="35.2679" y2="11.1379" width="0.508" layer="1"/>
+<wire x1="35.2679" y1="11.1379" x2="39.37" y2="15.24" width="0.508" layer="1"/>
+<wire x1="39.37" y1="15.24" x2="39.37" y2="17.145" width="0.508" layer="1"/>
+</signal>
 </signals>
